File: 01_PCB/Dori.sch (KiCad schematic (older format))
At the start: 200 parts, among them J1 TYPE-C-31-M12_13, J2 AVR-ISP-6_mod, J3 4PIN, J4 4PIN, J5 TYPE-C-31-M12_13, J6 AVR-ISP-6_mod, K1 KEYSW, K10 KEYSW, K11 KEYSW, K12 KEYSW, K13 KEYSW, K14 KEYSW, K15 KEYSW, K16 KEYSW, K17 KEYSW, K18 KEYSW, K19 KEYSW, K2 KEYSW, K20 KEYSW, K21 KEYSW, K22 KEYSW, K23 KEYSW, K24 KEYSW, K25 KEYSW, K26 KEYSW, K27 KEYSW, K28 KEYSW, K29 KEYSW, K3 KEYSW, K30 KEYSW, K31 KEYSW, K32 KEYSW, K33 KEYSW, K34 KEYSW, K35 KEYSW, K36 KEYSW, K37 KEYSW, K38 KEYSW, K39 KEYSW, K4 KEYSW, K40 KEYSW, K41 KEYSW, K42 KEYSW, K43 KEYSW, K44 KEYSW, K45 KEYSW, K46 KEYSW, K47 KEYSW, K48 KEYSW, K49 KEYSW, K5 KEYSW, K50 KEYSW, K51 KEYSW, K52 KEYSW, K53 KEYSW, K54 KEYSW, K55 KEYSW, K56 KEYSW, K6 KEYSW, K7 KEYSW, K8 KEYSW, K9 KEYSW, SW1 SW_PUSH, SW10 Rotary_Encoder_Switch, SW2 SW_PUSH, SW3 Rotary_Encoder_Switch, SW4 Rotary_Encoder_Switch, SW5 Rotary_Encoder_Switch, SW6 Rotary_Encoder_Switch, SW7 Rotary_Encoder_Switch, SW8 Rotary_Encoder_Switch, SW9 Rotary_Encoder_Switch, U1 ATMEGA32U4, U10 HOLE, U11 HOLE, U12 ATMEGA32U4, U13 HOLE, U14 HOLE, U15 HOLE, U16 HOLE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

Commit message: Update Dori.sch
Parts:
- added C13, C14: 4.7nF, Capacitor_SMD:C_0805_2012Metric_Pad1.15x1.40mm_HandSolder, symbol Device:C_Small
- added CESD1, CESD2: 100nF, Capacitor_SMD:C_0805_2012Metric_Pad1.15x1.40mm_HandSolder, symbol Device:C_Small
- added R15, R16: 1M, Resistor_SMD:R_0805_2012Metric_Pad1.15x1.40mm_HandSolder, symbol Device:R_Small
- F1, F2: value 500mA -> .5A
Connections:
- net GND: now also C13.2, CESD1.1, R15.2; no longer J1.S (SHIELD)
- net GNDA: now also SW5.C, C14.2, CESD2.1, R16.2; no longer J5.S (SHIELD)
- net VBUSa: now also CESD1.2
- net VBUSb: now also CESD2.2
- new net: C13.1, J1.S (SHIELD), R15.1
- new net: C14.1, J5.S (SHIELD), R16.1
Other:
- note added: "Left half"
- note added: "Right half"
- moved on the sheet: C1, C10, C11, C2, C3, C4, C5, C7, C8, C9, CX1, CX2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

Commit message: Routed data lines as differential pair
Connections:
- net Da-: now reaches R2.1, U1.3 (D-)
- net Da+: now reaches R3.1, U1.4 (D+)
- net Db-: now reaches R10.1, U12.3 (D-)
- net Db+: now reaches R11.1, U12.4 (D+)
- net D+BUSa renamed DBUSa+
- net D+BUSb renamed DBUSb+
- net D+a: no longer names the net of R3.2, U3.4 (IO2)
- net D+b: no longer names the net of R11.2, U8.4 (IO2)
- net D-BUSa renamed DBUSa-
- net D-BUSb renamed DBUSb-
- net D-a: no longer names the net of R2.2, U3.6 (IO1)
- net D-b: no longer names the net of R10.2, U8.6 (IO1)
Other:
- moved on the sheet: C1, C10, C11, C12, C13, C14, C2, C3, C4, C5, C6, C7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
