File: 01_PCB/niko.kicad_pcb (KiCad board)
At the start: 2 copper layers, 254.8 x 106.8 mm, 144 parts, among them J1 TYPE-C-31-M12_13, J2 AVR-ISP-6_mod, K1 KEYSW, K10 KEYSW, K11 KEYSW, K12 KEYSW, K13 KEYSW, K14 KEYSW, K15 KEYSW, K16 KEYSW, K17 KEYSW, K18 KEYSW, K19 KEYSW, K2 KEYSW, K20 KEYSW, K21 KEYSW, K22 KEYSW, K23 KEYSW, K24 KEYSW, K25 KEYSW, K26 KEYSW, K27 KEYSW, K28 KEYSW, K29 KEYSW, K3 KEYSW, K30 KEYSW, K31 KEYSW, K32 KEYSW, K33 KEYSW, K34 KEYSW, K35 KEYSW, K36 KEYSW, K37 KEYSW, K38 KEYSW, K39 KEYSW, K4 KEYSW, K40 KEYSW, K41 KEYSW, K42 KEYSW, K43 KEYSW, K44 KEYSW, K45 KEYSW, K46 KEYSW, K47 KEYSW, K48 KEYSW, K49 KEYSW, K5 KEYSW, K50 KEYSW, K51 KEYSW, K52 KEYSW, K53 KEYSW, K54 KEYSW, K55 KEYSW, K56 KEYSW, K57 KEYSW, K58 KEYSW, K59 KEYSW, K6 KEYSW, K60 KEYSW, K7 KEYSW, K8 KEYSW, K9 KEYSW, SW1 SW_PUSH, SW2 Rotary_Encoder_Switch, U1 ATMEGA32U4, U3 PRTR5V0U2X, Y1 16MHz

Commit message: start top plate
Routing:
- net col1: track 196.7 -> 200.7 mm
- net row0: track 388.2 -> 391.7 mm, vias 4 -> 2
- net ISP_RST: track 149.2 -> 148.5 mm

Commit message: made thumb buttons 1.5u
Parts:
- K42, K43: footprint Keeb_footprints:MX100 -> Keeb_footprints:MX_PCB_150H
- moved K44 9.55 mm to (290.5, 109.5)
- moved D12 9.53 mm to (365.9, 47.2)
- moved D24 9.53 mm to (365.9, 76.6)
- moved D36 9.53 mm to (365.9, 85.4)
- moved D48 9.53 mm to (365.9, 104.4)
- moved D60 9.53 mm to (365.9, 38.5)
- moved K20 9.53 mm to (297.6, 67.9)
- moved K32 9.53 mm to (297.6, 86.9)
- moved K57 9.53 mm to (316.7, 27.3)
- moved K8 9.53 mm to (297.6, 48.8)
- moved D10 9.53 mm to (327.8, 43.7)
- moved D11 9.53 mm to (362.8, 47.2)
- moved D19 9.53 mm to (286.5, 73.0)
- moved D20 9.53 mm to (289.7, 73.0)
- moved D21 9.53 mm to (324.6, 73.0)
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Routing:
- net row2: track 346.1 -> 365.1 mm
- net row3: track 386.8 -> 405.9 mm
- net row4: track 404.1 -> 423.1 mm
- net Net-(D44-Pad2): track 11.8 -> 22.4 mm
- net col11: track 193.5 -> 203.2 mm
- net col8: track 142.1 -> 151.6 mm
- net col10: track 175.2 -> 184.7 mm
- net col9: track 159.7 -> 169.3 mm
- net col7: track 129.8 -> 139.3 mm
- net row1: track 384.8 -> 394.3 mm
- net col6: track 101.7 -> 108.6 mm
- net row0: track 391.7 -> 397.9 mm, vias 2 -> 4
- net ISP_RST: track 148.5 -> 154.4 mm
- net D-: track 43.1 -> 48.0 mm
- net D+: track 42.3 -> 47.2 mm
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Other:
- board size 254.8 x 106.8 mm -> 264.3 x 111.6 mm
