File: 01_PCB/niko.sch (KiCad schematic (older format))
At the start: 144 parts, among them J1 TYPE-C-31-M12_13, J2 AVR-ISP-6_mod, K1 KEYSW, K10 KEYSW, K11 KEYSW, K12 KEYSW, K13 KEYSW, K14 KEYSW, K15 KEYSW, K16 KEYSW, K17 KEYSW, K18 KEYSW, K19 KEYSW, K2 KEYSW, K20 KEYSW, K21 KEYSW, K22 KEYSW, K23 KEYSW, K24 KEYSW, K25 KEYSW, K26 KEYSW, K27 KEYSW, K28 KEYSW, K29 KEYSW, K3 KEYSW, K30 KEYSW, K31 KEYSW, K32 KEYSW, K33 KEYSW, K34 KEYSW, K35 KEYSW, K36 KEYSW, K37 KEYSW, K38 KEYSW, K39 KEYSW, K4 KEYSW, K40 KEYSW, K41 KEYSW, K42 KEYSW, K43 KEYSW, K44 KEYSW, K45 KEYSW, K46 KEYSW, K47 KEYSW, K48 KEYSW, K49 KEYSW, K5 KEYSW, K50 KEYSW, K51 KEYSW, K52 KEYSW, K53 KEYSW, K54 KEYSW, K55 KEYSW, K56 KEYSW, K57 KEYSW, K58 KEYSW, K59 KEYSW, K6 KEYSW, K60 KEYSW, K7 KEYSW, K8 KEYSW, K9 KEYSW, SW1 SW_PUSH, SW2 Rotary_Encoder_Switch, U1 ATMEGA32U4, U3 PRTR5V0U2X, Y1 16MHz

Commit message: start top plate
Parts:
- J2: symbol niko_ergo-rescue:AVR-ISP-6_mod-Connector-Dori_Ergo-rescue -> niko-rescue:AVR-ISP-6_mod-Connector-Dori_Ergo-rescue-niko_ergo-rescue
Connections:
- net Enc0a: now also U1.31 (PC6)
- net Enc0b: now also U1.30 (PB6)
- net col1: now also U1.41 (PF0); no longer U1.42 (AREF)
- net col10: now also U1.21 (PD3/TXD1)
- net col11: now also U1.22 (PD5/XCK1)
- net col12: now also U1.32 (PC7); no longer U1.37 (PF6)
- net col2: now also U1.40 (PF1); no longer U1.41 (PF0)
- net col3: now also U1.39 (PF4); no longer U1.40 (PF1)
- net col4: now also U1.38 (PF5); no longer U1.39 (PF4)
- net col5: now also U1.37 (PF6); no longer U1.38 (PF5)
- net col6: now also U1.29 (PB5)
- net col7: now also U1.18 (PD0/INT0)
- net col8: now also U1.19 (PD1/INT1)
- net col9: now also U1.20 (PD2/RXD1)
- net row2: now also U1.27 (T0/PD7)
- net row3: now also U1.26 (T1/PD6)
- net row4: now also U1.25 (ICP1/PD4)
Changed lines of the file:
@@
 EESchema Schematic File Version 4
-LIBS:niko_ergo-cache
+LIBS:niko-cache
 EELAYER 30 0
 EELAYER END
@@
 Text GLabel 7450 8500 0    50   Output ~ 0
 row1
-Text GLabel 9600 7700 2    50   Output ~ 0
-col1
 Text GLabel 9600 7800 2    50   Output ~ 0
+col1
+Text GLabel 9600 7900 2    50   Output ~ 0
 col2
 $Comp
@@
 	0    1    1    0
 $EndComp
-Text GLabel 9600 8100 2    50   Output ~ 0
+Text GLabel 9600 8200 2    50   Output ~ 0
 col5
 $Comp
@@
 Text GLabel 7450 7700 0    50   Input ~ 0
 D-
-Text GLabel 10900 8100 2    50   Output ~ 0
+Text GLabel 9600 9300 2    50   Output ~ 0
 row3
 $Comp
@@
 col5
 $Comp
-L niko_ergo-rescue:AVR-ISP-6_mod-Connector-Dori_Ergo-rescue J2
+L niko-rescue:AVR-ISP-6_mod-Connector-Dori_Ergo-rescue-niko_ergo-rescue J2
 U 1 1 5EC10E7A
 P 8100 10650
@@
 Wire Notes Line
 	4500 12150 4500 11700
-Text GLabel 10900 8700 2    50   Output ~ 0
+Text GLabel 9600 8900 2    50   Output ~ 0
 Enc0b
-Text GLabel 10900 8600 2    50   Output ~ 0
+Text GLabel 9600 8800 2    50   Output ~ 0
 Enc0a
 Text GLabel 7450 8300 0    50   Output ~ 0
@@
 Text GLabel 7450 8400 0    50   Output ~ 0
 row0
-Text GLabel 9600 7900 2    50   Output ~ 0
+Text GLabel 9600 8000 2    50   Output ~ 0
 col3
-Text GLabel 10900 8400 2    50   Output ~ 0
+Text GLabel 9600 9200 2    50   Output ~ 0
 row2
-Text GLabel 9600 8000 2    50   Output ~ 0
+Text GLabel 9600 8100 2    50   Output ~ 0
 col4
 $Comp
@@
 Connection ~ 8900 2950
 Connection ~ 8200 6050
-Text GLabel 10900 8900 2    50   Output ~ 0
-Enc1b
-Text GLabel 10900 8800 2    50   Output ~ 0
-Enc1a
 $Comp
 L power:VCC #PWR0128
@@
 Text GLabel 8100 11050 3    50   Output ~ 0
 row1
-Text GLabel 10900 9100 2    50   Output ~ 0
+Text GLabel 7450 9200 0    50   Output ~ 0
 col7
-Text GLabel 10900 9000 2    50   Output ~ 0
+Text GLabel 9600 9000 2    50   Output ~ 0
 col6
-Text GLabel 10900 9200 2    50   Output ~ 0
+Text GLabel 7450 9300 0    50   Output ~ 0
 col8
-Text GLabel 10900 9300 2    50   Output ~ 0
+Text GLabel 7450 9400 0    50   Output ~ 0
 col9
-Text GLabel 10900 9400 2    50   Output ~ 0
+Text GLabel 7450 9500 0    50   Output ~ 0
 col10
-Text GLabel 10900 9500 2    50   Output ~ 0
+Text GLabel 7450 9600 0    50   Output ~ 0
 col11
-Text GLabel 9600 8200 2    50   Output ~ 0
+Text GLabel 9600 8700 2    50   Output ~ 0
 col12
 Text GLabel 9000 6700 0    50   Output ~ 0
 col12
+Text GLabel 9600 9400 2    50   Output ~ 0
+row4
 $EndSCHEMATC

Commit message: made thumb buttons 1.5u
Parts:
- K42, K43: footprint Keeb_footprints:MX100 -> Keeb_footprints:MX_PCB_150H
Changed lines of the file:
@@
 F 0 "K42" H 8550 5700 60  0000 C CNN
 F 1 "KEYSW" H 8550 5600 60  0001 C CNN
-F 2 "Keeb_footprints:MX100" H 8550 5700 60  0001 C CNN
+F 2 "Keeb_footprints:MX_PCB_150H" H 8550 5700 60  0001 C CNN
 F 3 "" H 8550 5700 60  0000 C CNN
 	1    8550 5700
@@
 F 0 "K43" H 10050 5700 60  0000 C CNN
 F 1 "KEYSW" H 10050 5600 60  0001 C CNN
-F 2 "Keeb_footprints:MX100" H 10050 5700 60  0001 C CNN
+F 2 "Keeb_footprints:MX_PCB_150H" H 10050 5700 60  0001 C CNN
 F 3 "" H 10050 5700 60  0000 C CNN
 	1    10050 5700
