File: 02_top_plate/niko_top_plate.kicad_pcb (KiCad board)
At the start: 2 copper layers, 257.2 x 113.1 mm, 69 parts, among them U1 HOLE, U10 HOLE, U11 HOLE, U12 HOLE, U13 HOLE, U14 HOLE, U15 HOLE, U16 HOLE, U17 HOLE, U18 HOLE, U19 HOLE, U2 HOLE, U20 HOLE, U21 HOLE, U22 HOLE, U23 HOLE, U24 HOLE, U25 HOLE, U26 HOLE, U27 HOLE, U28 HOLE, U29 HOLE, U3 HOLE, U30 HOLE, U31 HOLE, U32 HOLE, U33 HOLE, U34 HOLE, U35 HOLE, U36 HOLE, U37 HOLE, U38 HOLE, U39 HOLE, U4 HOLE, U40 HOLE, U41 HOLE, U42 HOLE, U43 HOLE, U44 HOLE, U45 HOLE, U46 HOLE, U47 HOLE, U48 HOLE, U49 HOLE, U5 HOLE, U50 HOLE, U51 HOLE, U52 HOLE, U53 HOLE, U54 HOLE, U55 HOLE, U56 HOLE, U57 HOLE, U58 HOLE, U59 HOLE, U6 HOLE, U60 HOLE, U7 HOLE, U8 HOLE, U9 HOLE

Commit message: finish top plate; add bottom plate
Parts:
- added U61: HOLE, Keeb_footprints:MX100_cutout_plated, F.Cu at (192.9, 146.4)
- moved H4 8.67 mm to (161.9, 179.8)
- moved H8 0.60 mm to (311.9, 178.0)
- moved H1 0.60 mm to (73.8, 79.2)
- moved H2 0.60 mm to (73.8, 178.0)
- moved H3 0.60 mm to (150.0, 73.2)
- moved H5 0.60 mm to (235.7, 73.2)
- moved H7 0.60 mm to (311.9, 79.2)
Routing:
- added copper zone on B.Cu, net (none)
- added copper zone on F.Cu, net GND
Other:
- board size 257.2 x 113.1 mm -> 257.2 x 112.5 mm
