File: 02_top_plate/top_plate.kicad_pcb (KiCad board)
At the start: 2 copper layers, 257.2 x 112.5 mm, 70 parts, among them U1 HOLE, U10 HOLE, U11 HOLE, U12 HOLE, U13 HOLE, U14 HOLE, U15 HOLE, U16 HOLE, U17 HOLE, U18 HOLE, U19 HOLE, U2 HOLE, U20 HOLE, U21 HOLE, U22 HOLE, U23 HOLE, U24 HOLE, U25 HOLE, U26 HOLE, U27 HOLE, U28 HOLE, U29 HOLE, U3 HOLE, U30 HOLE, U31 HOLE, U32 HOLE, U33 HOLE, U34 HOLE, U35 HOLE, U36 HOLE, U37 HOLE, U38 HOLE, U39 HOLE, U4 HOLE, U40 HOLE, U41 HOLE, U42 HOLE, U43 HOLE, U44 HOLE, U45 HOLE, U46 HOLE, U47 HOLE, U48 HOLE, U49 HOLE, U5 HOLE, U50 HOLE, U51 HOLE, U52 HOLE, U53 HOLE, U54 HOLE, U55 HOLE, U56 HOLE, U57 HOLE, U58 HOLE, U59 HOLE, U6 HOLE, U60 HOLE, U61 HOLE, U7 HOLE, U8 HOLE, U9 HOLE

Commit message: remove 4 keys
Parts:
- removed D2: DIODE, Keeb_footprints:D_SOD-123_modified
- removed U37, U38, U47, U48: HOLE, Keeb_footprints:MX100_cutout_plated
- added R1: R_Small, Resistor_SMD:R_0603_1608Metric_Pad1.05x0.95mm_HandSolder, B.Cu at (321.5, 100.0)
- U42, U43: footprint Keeb_footprints:MX100_cutout_plated -> Keeb_footprints:MX_150_cutout_plated
- moved H8 21.3 mm to (321.5, 158.9)
- moved H2 19.1 mm to (73.8, 158.9)
- moved H6 17.4 mm to (241.1, 178.0)
- moved H7 9.53 mm to (321.5, 79.2)
- moved U11 9.53 mm to (302.4, 109.5)
- moved U23 9.53 mm to (302.4, 128.6)
- moved U35 9.53 mm to (302.4, 147.6)
- moved U59 9.53 mm to (302.4, 90.5)
- moved U21 9.53 mm to (264.3, 122.6)
- moved U33 9.53 mm to (264.3, 141.7)
- moved U44 9.53 mm to (238.1, 166.7)
- moved U45 9.53 mm to (264.3, 160.7)
- moved U57 9.53 mm to (264.3, 84.5)
- moved U9 9.53 mm to (264.3, 103.6)
- moved H5 9.53 mm to (245.3, 73.2)
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Routing:
- net (no net): track 2.52 -> 0.00 mm, vias 1 -> 0
- net GND: track 0.00 -> 1.51 mm, vias 0 -> 1
Other:
- board size 257.2 x 112.5 mm -> 266.7 x 118.2 mm
