File: 01_pcb/pcb.sch (KiCad schematic (older format))
At the start: 144 parts, among them J1 TYPE-C-31-M12_13, J2 AVR-ISP-6_mod, K1 KEYSW, K10 KEYSW, K11 KEYSW, K12 KEYSW, K13 KEYSW, K14 KEYSW, K15 KEYSW, K16 KEYSW, K17 KEYSW, K18 KEYSW, K19 KEYSW, K2 KEYSW, K20 KEYSW, K21 KEYSW, K22 KEYSW, K23 KEYSW, K24 KEYSW, K25 KEYSW, K26 KEYSW, K27 KEYSW, K28 KEYSW, K29 KEYSW, K3 KEYSW, K30 KEYSW, K31 KEYSW, K32 KEYSW, K33 KEYSW, K34 KEYSW, K35 KEYSW, K36 KEYSW, K37 KEYSW, K38 KEYSW, K39 KEYSW, K4 KEYSW, K40 KEYSW, K41 KEYSW, K42 KEYSW, K43 KEYSW, K44 KEYSW, K45 KEYSW, K46 KEYSW, K47 KEYSW, K48 KEYSW, K49 KEYSW, K5 KEYSW, K50 KEYSW, K51 KEYSW, K52 KEYSW, K53 KEYSW, K54 KEYSW, K55 KEYSW, K56 KEYSW, K57 KEYSW, K58 KEYSW, K59 KEYSW, K6 KEYSW, K60 KEYSW, K7 KEYSW, K8 KEYSW, K9 KEYSW, SW1 SW_PUSH, SW2 Rotary_Encoder_Switch, U1 ATMEGA32U4, U3 PRTR5V0U2X, Y1 16MHz

Commit message: rename files; reborder pcb
Parts:
- removed D37, D38, D47, D48: D, Keeb_footprints:D_SOD-123_modified, symbol keyboard_parts:D
- removed K37, K38, K47, K48: KEYSW, Keeb_footprints:MX100, symbol keyboard_parts:KEYSW
- J2: symbol niko-rescue:AVR-ISP-6_mod-Connector-Dori_Ergo-rescue-niko_ergo-rescue -> pcb-rescue:AVR-ISP-6_mod-Connector-Dori_Ergo-rescue-niko_ergo-rescue-niko-rescue
- K42, K43: footprint Keeb_footprints:MX100 -> Keeb_footprints:MX_PCB_150H
Connections:
- wire segments 427 -> 403
Changed lines of the file:
@@
 EESchema Schematic File Version 4
-LIBS:niko-cache
+LIBS:pcb-cache
 EELAYER 30 0
 EELAYER END
@@
 Wire Wire Line
 	4800 5300 4800 5350
-Connection ~ 4650 5000
-Connection ~ 5500 5000
 Connection ~ 6350 5000
 Connection ~ 7200 5000
@@
 Connection ~ 8900 5000
 Wire Wire Line
-	4800 6050 5650 6050
-Connection ~ 4800 6050
-Wire Wire Line
-	4800 6000 4800 6050
-Wire Wire Line
 	5650 6050 6500 6050
-Connection ~ 5650 6050
 Wire Wire Line
 	5650 6000 5650 6050
@@
 	8200 6000 8200 6050
 Wire Wire Line
-	3950 6050 4800 6050
-Wire Wire Line
-	3950 6000 3950 6050
-Wire Wire Line
 	8900 5000 8900 5700
 Wire Wire Line
@@
 Wire Wire Line
 	6350 5000 6350 5700
-Wire Wire Line
-	5500 5000 5500 5700
-Wire Wire Line
-	4650 5000 4650 5700
 Wire Wire Line
 	8200 5700 8200 5800
@@
 F 0 "K42" H 8550 5700 60  0000 C CNN
 F 1 "KEYSW" H 8550 5600 60  0001 C CNN
-F 2 "Keeb_footprints:MX100" H 8550 5700 60  0001 C CNN
+F 2 "Keeb_footprints:MX_PCB_150H" H 8550 5700 60  0001 C CNN
 F 3 "" H 8550 5700 60  0000 C CNN
 	1    8550 5700
@@
 F 3 "" H 6000 5700 60  0000 C CNN
 	1    6000 5700
-	1    0    0    -1
-$EndComp
-Wire Wire Line
-	4800 5700 4800 5800
-Wire Wire Line
-	4850 5700 4800 5700
-$Comp
-L keyboard_parts:D D38
-U 1 1 5DBF7BD0
-P 4800 5950
-F 0 "D38" H 4672 5900 60  0000 R CNN
-F 1 "D" V 4950 5900 60  0001 C CNN
-F 2 "Keeb_footprints:D_SOD-123_modified" H 4800 5950 60  0001 C CNN
-F 3 "" H 4800 5950 60  0000 C CNN
-	1    4800 5950
-	-1   0    0    1
-$EndComp
-Wire Wire Line
-	5500 5700 5450 5700
-$Comp
-L keyboard_parts:KEYSW K38
-U 1 1 5DBF7BD7
-P 5150 5700
-F 0 "K38" H 5150 5700 60  0000 C CNN
-F 1 "KEYSW" H 5150 5600 60  0001 C CNN
-F 2 "Keeb_footprints:MX100" H 5150 5700 60  0001 C CNN
-F 3 "" H 5150 5700 60  0000 C CNN
-	1    5150 5700
-	1    0    0    -1
-$EndComp
-Wire Wire Line
-	3950 5700 3950 5800
-Wire Wire Line
-	4000 5700 3950 5700
-$Comp
-L keyboard_parts:D D37
-U 1 1 5DBF7BDF
-P 3950 5950
-F 0 "D37" H 3822 5900 60  0000 R CNN
-F 1 "D" V 4100 5900 60  0001 C CNN
-F 2 "Keeb_footprints:D_SOD-123_modified" H 3950 5950 60  0001 C CNN
-F 3 "" H 3950 5950 60  0000 C CNN
-	1    3950 5950
-	-1   0    0    1
-$EndComp
-Wire Wire Line
-	4650 5700 4600 5700
-$Comp
-L keyboard_parts:KEYSW K37
-U 1 1 5DBF7BE6
-P 4300 5700
-F 0 "K37" H 4300 5700 60  0000 C CNN
-F 1 "KEYSW" H 4300 5600 60  0001 C CNN
-F 2 "Keeb_footprints:MX100" H 4300 5700 60  0001 C CNN
-F 3 "" H 4300 5700 60  0000 C CNN
-	1    4300 5700
 	1    0    0    -1
 $EndComp
@@
 col5
 $Comp
-L niko-rescue:AVR-ISP-6_mod-Connector-Dori_Ergo-rescue-niko_ergo-rescue J2
+L pcb-rescue:AVR-ISP-6_mod-Connector-Dori_Ergo-rescue-niko_ergo-rescue-niko-rescue J2
 U 1 1 5EC10E7A
 P 8100 10650
@@
 F 0 "K43" H 10050 5700 60  0000 C CNN
 F 1 "KEYSW" H 10050 5600 60  0001 C CNN
-F 2 "Keeb_footprints:MX100" H 10050 5700 60  0001 C CNN
+F 2 "Keeb_footprints:MX_PCB_150H" H 10050 5700 60  0001 C CNN
 F 3 "" H 10050 5700 60  0000 C CNN
 	1    10050 5700
@@
 Wire Wire Line
 	12250 5700 12250 5800
-$Comp
-L keyboard_parts:KEYSW K47
-U 1 1 5DBF7B50
-P 13450 5700
-F 0 "K47" H 13450 5700 60  0000 C CNN
-F 1 "KEYSW" H 13450 5600 60  0001 C CNN
-F 2 "Keeb_footprints:MX100" H 13450 5700 60  0001 C CNN
-F 3 "" H 13450 5700 60  0000 C CNN
-	1    13450 5700
-	1    0    0    -1
-$EndComp
-Wire Wire Line
-	13800 5700 13750 5700
-$Comp
-L keyboard_parts:D D47
-U 1 1 5DBF7B49
-P 13100 5950
-F 0 "D47" H 12972 5900 60  0000 R CNN
-F 1 "D" V 13250 5900 60  0001 C CNN
-F 2 "Keeb_footprints:D_SOD-123_modified" H 13100 5950 60  0001 C CNN
-F 3 "" H 13100 5950 60  0000 C CNN
-	1    13100 5950
-	-1   0    0    1
-$EndComp
-Wire Wire Line
-	13150 5700 13100 5700
-Wire Wire Line
-	13100 5700 13100 5800
-$Comp
-L keyboard_parts:KEYSW K48
-U 1 1 5DBF7B41
-P 14300 5700
-F 0 "K48" H 14300 5700 60  0000 C CNN
-F 1 "KEYSW" H 14300 5600 60  0001 C CNN
-F 2 "Keeb_footprints:MX100" H 14300 5700 60  0001 C CNN
-F 3 "" H 14300 5700 60  0000 C CNN
-	1    14300 5700
-	1    0    0    -1
-$EndComp
-$Comp
-L keyboard_parts:D D48
-U 1 1 5DBF7B3A
-P 13950 5950
-F 0 "D48" H 13822 5900 60  0000 R CNN
-F 1 "D" V 14100 5900 60  0001 C CNN
-F 2 "Keeb_footprints:D_SOD-123_modified" H 13950 5950 60  0001 C CNN
-F 3 "" H 13950 5950 60  0000 C CNN
-	1    13950 5950
-	-1   0    0    1
-$EndComp
-Wire Wire Line
-	14000 5700 13950 5700
-Wire Wire Line
-	13950 5700 13950 5800
 Wire Wire Line
 	10400 5000 10400 5700
@@
 	12950 5000 12950 5700
 Wire Wire Line
-	13800 5000 13800 5700
-Wire Wire Line
-	13950 6050 13950 6000
-Wire Wire Line
-	13100 6000 13100 6050
-Connection ~ 13100 6050
-Wire Wire Line
-	13100 6050 13950 6050
-Wire Wire Line
 	12250 6000 12250 6050
-Connection ~ 12250 6050
-Wire Wire Line
-	12250 6050 13100 6050
 Wire Wire Line
 	11400 6000 11400 6050
@@
 Wire Wire Line
 	9700 6050 10550 6050
-Connection ~ 13800 5000
 Connection ~ 12950 5000
 Connection ~ 12100 5000
@@
 Wire Wire Line
 	14600 5000 14650 5000
-Connection ~ 14650 5000
-Wire Wire Line
-	14650 5000 14650 5700
-Wire Wire Line
-	14650 5700 14600 5700
 Wire Wire Line
 	14650 3600 14650 4300
@@
 Text GLabel 3800 6050 0    50   Input ~ 0
 row4
-Wire Wire Line
-	3950 6050 3800 6050
-Connection ~ 3950 6050
 Wire Wire Line
 	3950 4650 3800 4650
@@
 Text GLabel 9600 9400 2    50   Output ~ 0
 row4
+Wire Wire Line
+	5650 6050 3800 6050
+Connection ~ 5650 6050
 $EndSCHEMATC

Commit message: update gerber
Connections:
- net col1: now also SW2.S1
- net col12: no longer SW2.S1
- net row3: no longer D61.1
- net row4: now also D61.1
- no-connect marks 2 -> 8
Changed lines of the file:
@@
 	9000 6500 8600 6500
-Wire Wire Line
-	8200 5350 9100 5350
-Wire Wire Line
-	9100 5350 9100 6200
-Wire Wire Line
-	9100 6200 8400 6200
-Connection ~ 9100 5350
-Wire Wire Line
-	9100 5350 9700 5350
-Wire Wire Line
-	8600 6800 8400 6800
-Wire Wire Line
-	8400 6200 8400 6800
 Wire Wire Line
 	8600 6800 8600 6700
@@
 Text GLabel 9600 8700 2    50   Output ~ 0
 col12
-Text GLabel 9000 6700 0    50   Output ~ 0
-col12
 Text GLabel 9600 9400 2    50   Output ~ 0
 row4
 Wire Wire Line
-	5650 6050 3800 6050
+	5650 6050 5250 6050
 Connection ~ 5650 6050
+Wire Wire Line
+	5250 6800 5250 6050
+Connection ~ 5250 6050
+Wire Wire Line
+	5250 6050 3800 6050
+Wire Wire Line
+	5250 6800 8600 6800
+Wire Wire Line
+	8200 5350 9700 5350
+Wire Wire Line
+	5500 5000 5500 6900
+Wire Wire Line
+	5500 6900 8950 6900
+Wire Wire Line
+	8950 6900 8950 6700
+Wire Wire Line
+	8950 6700 9000 6700
+Connection ~ 5500 5000
+NoConn ~ 9600 7700
+NoConn ~ 9600 8300
+NoConn ~ 9600 9100
+NoConn ~ 7450 8600
+NoConn ~ 7450 8200
+NoConn ~ 7450 7500
 $EndSCHEMATC
