File: 01_pcb/pcb.kicad_pcb (KiCad board)
At the start: 2 copper layers, 264.3 x 111.6 mm, 144 parts, among them J1 TYPE-C-31-M12_13, J2 AVR-ISP-6_mod, K1 KEYSW, K10 KEYSW, K11 KEYSW, K12 KEYSW, K13 KEYSW, K14 KEYSW, K15 KEYSW, K16 KEYSW, K17 KEYSW, K18 KEYSW, K19 KEYSW, K2 KEYSW, K20 KEYSW, K21 KEYSW, K22 KEYSW, K23 KEYSW, K24 KEYSW, K25 KEYSW, K26 KEYSW, K27 KEYSW, K28 KEYSW, K29 KEYSW, K3 KEYSW, K30 KEYSW, K31 KEYSW, K32 KEYSW, K33 KEYSW, K34 KEYSW, K35 KEYSW, K36 KEYSW, K37 KEYSW, K38 KEYSW, K39 KEYSW, K4 KEYSW, K40 KEYSW, K41 KEYSW, K42 KEYSW, K43 KEYSW, K44 KEYSW, K45 KEYSW, K46 KEYSW, K47 KEYSW, K48 KEYSW, K49 KEYSW, K5 KEYSW, K50 KEYSW, K51 KEYSW, K52 KEYSW, K53 KEYSW, K54 KEYSW, K55 KEYSW, K56 KEYSW, K57 KEYSW, K58 KEYSW, K59 KEYSW, K6 KEYSW, K60 KEYSW, K7 KEYSW, K8 KEYSW, K9 KEYSW, SW1 SW_PUSH, SW2 Rotary_Encoder_Switch, U1 ATMEGA32U4, U3 PRTR5V0U2X, Y1 16MHz

Commit message: rename files; reborder pcb
Parts:
- removed D37, D38, D47, D48: D, Keeb_footprints:D_SOD-123_modified
- removed K37, K38, K47, K48: KEYSW, Keeb_footprints:MX100
Routing:
- net row4: track 423.1 -> 376.7 mm
- net col1: track 200.7 -> 181.6 mm
- net col0: track 207.1 -> 188.0 mm
- net col11: track 203.2 -> 184.2 mm
- net col10: track 184.7 -> 165.6 mm
- net Net-(D38-Pad2): track 11.2 -> 0.00 mm
- net Net-(D48-Pad2): track 11.1 -> 0.00 mm
- net Net-(D47-Pad2): track 6.14 -> 0.00 mm
- net Net-(D37-Pad2): track 6.11 -> 0.00 mm
Other:
- outline, holes or cut-outs redrawn

Commit message: remove 4 keys
Parts:
- moved K42 1.19 mm to (233.4, 114.3)
- moved K43 1.19 mm to (266.7, 114.3)
Other:
- outline, holes or cut-outs redrawn
Changed lines of the file:
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@@
     (thickness 1.6)
     (drawings 32)
-    (tracks 706)
+    (tracks 707)
     (zones 0)
     (modules 136)
@@
   )
   (module Keeb_footprints:MX_PCB_150H locked (layer F.Cu)
-    (at 232.17285 114.30048 60)
+    (at 233.36348 114.30048 60)
     (fp_text reference K42 (at 0 3.175 60) (layer Dwgs.User)
       (effects (font (size 1.27 1.524) (thickness 0.2032)))
@@
   )
   (module Keeb_footprints:MX_PCB_150H locked (layer F.Cu)
-    (at 267.89175 114.30048 300)
+    (at 266.70112 114.30048 300)
     (fp_text reference K43 (at 0 3.175 300) (layer Dwgs.User)
       (effects (font (size 1.27 1.524) (thickness 0.2032)))
@@
   (gr_line (start 198.83521 114.30048) (end 216.69466 120.25363) (layer Edge.Cuts) (width 0.05))
   (gr_line (start 172.64135 114.30048) (end 198.83521 114.30048) (layer Edge.Cuts) (width 0.05))
-  (gr_line (start 191.69143 19.05008) (end 210.74151 19.05008) (layer Edge.Cuts) (width 0.05))
+  (gr_line (start 173.83198 19.05008) (end 210.74151 19.05008) (layer Edge.Cuts) (width 0.05))
   (gr_line (start 289.32309 19.05008) (end 308.37317 19.05008) (layer Edge.Cuts) (width 0.05))
-  (gr_line (start 325.04199 19.05008) (end 379.81097 19.05008) (layer Edge.Cuts) (width 0.05))
+  (gr_line (start 326.23262 19.05008) (end 379.81097 25.00323) (layer Edge.Cuts) (width 0.05))
   (gr_line (start 301.22939 114.30048) (end 283.36994 120.25363) (layer Edge.Cuts) (width 0.05))
   (gr_line (start 327.42325 114.30048) (end 301.22939 114.30048) (layer Edge.Cuts) (width 0.05))
   (gr_arc (start 254.31252 19.05) (end 255.16252 19.05) (angle -90) (layer Edge.Cuts) (width 0.05))
-  (gr_line (start 354.80774 98.82229) (end 379.81097 98.82229) (layer Edge.Cuts) (width 0.05))
-  (gr_line (start 344.09207 114.30048) (end 354.80774 98.82229) (layer Edge.Cuts) (width 0.05))
+  (gr_line (start 355.99837 98.82229) (end 379.81097 98.82229) (layer Edge.Cuts) (width 0.05))
+  (gr_line (start 344.09207 114.30048) (end 355.99837 98.82229) (layer Edge.Cuts) (width 0.05))
   (gr_line (start 342.90144 114.30048) (end 344.09207 114.30048) (layer Edge.Cuts) (width 0.05))
   (gr_line (start 145.25686 98.82229) (end 120.25363 98.82229) (layer Edge.Cuts) (width 0.05))
   (gr_line (start 155.97253 114.30048) (end 145.25686 98.82229) (layer Edge.Cuts) (width 0.05))
   (gr_arc (start 379.81097 96.44103) (end 379.81097 98.82229) (angle -90) (layer Edge.Cuts) (width 0.05))
-  (gr_arc (start 379.81097 21.43134) (end 382.19223 21.43134) (angle -90) (layer Edge.Cuts) (width 0.05))
-  (gr_arc (start 120.25363 21.43134) (end 120.25363 19.05008) (angle -90) (layer Edge.Cuts) (width 0.05))
+  (gr_arc (start 379.81097 27.38449) (end 382.19223 27.38449) (angle -90) (layer Edge.Cuts) (width 0.05))
+  (gr_arc (start 120.25363 27.38449) (end 120.25363 25.00323) (angle -90) (layer Edge.Cuts) (width 0.05))
   (gr_arc (start 120.25363 96.44103) (end 117.87237 96.44103) (angle -90) (layer Edge.Cuts) (width 0.05))
   (gr_line (start 216.69466 120.25363) (end 233.36348 129.77867) (layer Edge.Cuts) (width 0.05))
@@
   (gr_arc (start 245.76252 19.05) (end 245.76252 18.2) (angle -90) (layer Edge.Cuts) (width 0.05))
   (gr_line (start 245.76252 18.2) (end 254.31252 18.2) (layer Edge.Cuts) (width 0.05))
-  (gr_line (start 120.25363 19.05008) (end 191.69143 19.05008) (layer Edge.Cuts) (width 0.05))
-  (gr_line (start 325.04199 19.05008) (end 308.37317 19.05008) (layer Edge.Cuts) (width 0.05))
-  (gr_line (start 382.19223 96.44103) (end 382.19223 21.43134) (layer Edge.Cuts) (width 0.05))
+  (gr_line (start 120.25363 25.00323) (end 173.83198 19.05008) (layer Edge.Cuts) (width 0.05))
+  (gr_line (start 326.23262 19.05008) (end 308.37317 19.05008) (layer Edge.Cuts) (width 0.05))
+  (gr_line (start 382.19223 96.44103) (end 382.19223 27.38449) (layer Edge.Cuts) (width 0.05))
   (gr_line (start 233.36348 129.77867) (end 266.70112 129.77867) (layer Edge.Cuts) (width 0.05))
-  (gr_line (start 117.87237 21.43134) (end 117.87237 96.44103) (layer Edge.Cuts) (width 0.05))
+  (gr_line (start 117.87237 27.38449) (end 117.87237 96.44103) (layer Edge.Cuts) (width 0.05))
   (gr_text "github.com/dierickdie\nniko rev 1.0" (at 250.0323 123.82552) (layer B.SilkS)
     (effects (font (size 1.25 1.25) (thickness 0.2)) (justify mirror))
@@
   (segment (start 215.357589 103.25) (end 213.319132 105.288457) (width 0.25) (layer B.Cu) (net 39))
   (segment (start 219.9 103.25) (end 215.357589 103.25) (width 0.25) (layer B.Cu) (net 39))
-  (segment (start 223.4 111.661892) (end 228.068145 116.330037) (width 0.25) (layer B.Cu) (net 40))
-  (segment (start 223.4 103.25) (end 223.4 111.661892) (width 0.25) (layer B.Cu) (net 40))
-  (segment (start 267.1 108.644468) (end 268.186455 109.730923) (width 0.25) (layer B.Cu) (net 41))
-  (segment (start 267.1 103.25) (end 267.1 108.644468) (width 0.25) (layer B.Cu) (net 41))
+  (segment (start 223.4 110.471262) (end 229.258775 116.330037) (width 0.25) (layer B.Cu) (net 40))
+  (segment (start 223.4 103.25) (end 223.4 110.471262) (width 0.25) (layer B.Cu) (net 40))
+  (segment (start 267.1 109.626748) (end 266.995825 109.730923) (width 0.25) (layer B.Cu) (net 41))
+  (segment (start 267.1 103.25) (end 267.1 109.626748) (width 0.25) (layer B.Cu) (net 41))
   (segment (start 290.928714 103.25) (end 291.65237 103.973656) (width 0.25) (layer B.Cu) (net 42))
   (segment (start 290.968803 103.25) (end 291.673618 103.954815) (width 0.25) (layer B.Cu) (net 42))
@@
   (segment (start 172.3 74.65) (end 140.904999 74.65) (width 0.25) (layer B.Cu) (net 57))
   (segment (start 175.4 74.65) (end 213.5 74.65) (width 0.25) (layer B.Cu) (net 57))
-  (segment (start 213.5 74.65) (end 277 74.65) (width 0.25) (layer B.Cu) (net 57))
-  (segment (start 286.52504 74.65) (end 277 74.65) (width 0.25) (layer B.Cu) (net 57))
   (segment (start 365.92504 77.1) (end 365.92504 78.25) (width 0.25) (layer B.Cu) (net 57))
   (segment (start 364.22504 75.4) (end 365.92504 77.1) (width 0.25) (layer B.Cu) (net 57))
@@
   (segment (start 361.21028 57.48524) (end 364.22504 60.5) (width 0.25) (layer B.Cu) (net 57))
   (segment (start 254.5 59.9) (end 255.78001 59.9) (width 0.25) (layer B.Cu) (net 57))
+  (segment (start 286.52504 74.65) (end 277 74.65) (width 0.25) (layer B.Cu) (net 57))
+  (segment (start 213.5 74.65) (end 277 74.65) (width 0.25) (layer B.Cu) (net 57))
   (segment (start 134.2 83.75) (end 137.3 83.75) (width 0.25) (layer B.Cu) (net 58))
   (segment (start 172.3 80.15) (end 175.375 80.15) (width 0.25) (layer B.Cu) (net 58))
@@
   (segment (start 321.67504 77.2) (end 292.67504 77.2) (width 0.25) (layer B.Cu) (net 58))
   (segment (start 324.62504 80.15) (end 321.67504 77.2) (width 0.25) (layer B.Cu) (net 58))
-  (segment (start 281.76252 80.15) (end 286.52504 80.15) (width 0.25) (layer B.Cu) (net 58))
-  (segment (start 213.5 80.15) (end 281.76252 80.15) (width 0.25) (layer B.Cu) (net 58))
   (segment (start 368.59503 81.08001) (end 365.92504 83.75) (width 0.25) (layer B.Cu) (net 58))
   (segment (start 378.58501 81.08001) (end 368.59503 81.08001) (width 0.25) (layer B.Cu) (net 58))
@@
   (segment (start 380.24503 59.657404) (end 380.24503 79.41999) (width 0.25) (layer B.Cu) (net 58))
   (segment (start 254.5 59.1) (end 262.237415 59.1) (width 0.25) (layer B.Cu) (net 58))
+  (segment (start 281.76252 80.15) (end 286.52504 80.15) (width 0.25) (layer B.Cu) (net 58))
+  (segment (start 213.5 80.15) (end 281.76252 80.15) (width 0.25) (layer B.Cu) (net 58))
   (segment (start 128.74678 28.25764) (end 132.95764 28.25764) (width 0.25) (layer B.Cu) (net 59))
   (segment (start 134.2 29.5) (end 132.95764 28.25764) (width 0.25) (layer B.Cu) (net 59))
@@
   (segment (start 250.2 67.8) (end 249.36002 68.63998) (width 0.25) (layer B.Cu) (net 78))
   (segment (start 250.2 66.6) (end 250.2 67.8) (width 0.25) (layer B.Cu) (net 78))
-  (segment (start 217.64625 98.163584) (end 229.043441 109.560775) (width 0.25) (layer F.Cu) (net 78))
-  (segment (start 217.64625 86.75725) (end 217.64625 98.163584) (width 0.25) (layer F.Cu) (net 78))
+  (segment (start 217.64625 96.972954) (end 230.234071 109.560775) (width 0.25) (layer F.Cu) (net 78))
+  (segment (start 217.64625 86.75725) (end 217.64625 96.972954) (width 0.25) (layer F.Cu) (net 78))
   (segment (start 262.76002 65.19594) (end 265.27125 67.70717) (width 0.25) (layer B.Cu) (net 79))
   (segment (start 262.76002 63.68519) (end 262.76002 65.19594) (width 0.25) (layer B.Cu) (net 79))
@@
   (segment (start 274.79629 86.75725) (end 274.79629 29.60814) (width 0.25) (layer F.Cu) (net 79))
   (segment (start 274.79629 67.70717) (end 265.27125 67.70717) (width 0.25) (layer B.Cu) (net 79))
-  (segment (start 274.79629 112.725054) (end 273.561159 113.960185) (width 0.25) (layer F.Cu) (net 79))
-  (segment (start 274.79629 86.75725) (end 274.79629 112.725054) (width 0.25) (layer F.Cu) (net 79))
+  (segment (start 274.79629 111.534424) (end 272.370529 113.960185) (width 0.25) (layer F.Cu) (net 79))
+  (segment (start 274.79629 107.89629) (end 274.79629 111.534424) (width 0.25) (layer F.Cu) (net 79))
+  (segment (start 274.79629 86.75725) (end 274.79629 107.89629) (width 0.25) (layer F.Cu) (net 79))
   (segment (start 293.8475 84.36208) (end 293.84629 84.36329) (width 0.25) (layer F.Cu) (net 80))
   (segment (start 293.8475 27.22575) (end 293.8475 84.36208) (width 0.25) (layer F.Cu) (net 80))
@@
     (polygon
       (pts
-        (xy 107.1567 11.9063) (xy 107.1567 130.9693) (xy 392.9079 130.9693) (xy 392.9079 11.9063)
+        (xy 107.1567 11.9063) (xy 107.1567 134.54119) (xy 392.9079 134.54119) (xy 392.9079 11.9063)
       )
     )
@@
     (polygon
       (pts
-        (xy 392.9079 11.9063) (xy 392.9079 130.9693) (xy 107.1567 130.9693) (xy 107.1567 11.9063)
+        (xy 392.9079 11.9063) (xy 392.9079 134.54119) (xy 107.1567 134.54119) (xy 107.1567 11.9063)
       )
     )

Commit message: update gerber
Connections:
- D61 pad 1: row3 -> row4
- SW2 pad S1: col12 -> col1
- U1 pad 32: col12 -> (no net)
Routing:
- net col1: track 181.6 -> 308.9 mm
- net col12: track 43.2 -> 0.00 mm, vias 1 -> 0
- net row4: track 376.7 -> 399.8 mm
- net row3: track 405.9 -> 407.8 mm
Changed lines of the file:
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@@
     (thickness 1.6)
     (drawings 32)
-    (tracks 707)
+    (tracks 714)
     (zones 0)
     (modules 136)
-    (nets 93)
+    (nets 92)
   )
   (page A3)
@@
     (solder_mask_min_width 0.25)
     (aux_axis_origin 245.26875 79.375)
-    (visible_elements 7FFFFFFF)
+    (visible_elements 7FFFEFFF)
     (pcbplotparams
       (layerselection 0x010fc_ffffffff)
@@
   (net 90 row4)
   (net 91 "Net-(D61-Pad2)")
-  (net 92 col12)
   (net_class Default "This is the default net class."
     (clearance 0.13)
@@
     (add_net col10)
     (add_net col11)
-    (add_net col12)
     (add_net col2)
     (add_net col3)
@@
       (net 91 "Net-(D61-Pad2)"))
     (pad 1 smd roundrect (at -1.65 0 270) (size 1 1.2) (layers B.Cu B.Paste B.Mask) (roundrect_rratio 0.25)
-      (net 58 row3))
+      (net 90 row4))
     (model ${KISYS3DMOD}/Diode_SMD.3dshapes/D_SOD-123.wrl
       (at (xyz 0 0 0))
@@
     (fp_line (start -7.8 -4.1) (end -7.2 -4.1) (layer B.SilkS) (width 0.12))
     (pad S1 thru_hole circle (at 7 2.5) (size 2 2) (drill 1) (layers *.Cu *.Mask)
-      (net 92 col12))
+      (net 74 col1))
     (pad S2 thru_hole circle (at 7 -2.5) (size 2 2) (drill 1) (layers *.Cu *.Mask)
       (net 91 "Net-(D61-Pad2)"))
@@
       (net 51 Enc0a) (solder_mask_margin 0.2))
     (pad 32 smd rect (at 5.9 3.2) (size 1.5 0.5) (layers B.Cu B.Paste B.Mask)
-      (net 92 col12) (solder_mask_margin 0.2))
+      (solder_mask_margin 0.2))
     (pad 33 smd rect (at 5.9 4) (size 1.5 0.5) (layers B.Cu B.Paste B.Mask)
       (net 46 "Net-(R1-Pad2)") (solder_mask_margin 0.2))
@@
   (segment (start 380.24503 59.657404) (end 380.24503 79.41999) (width 0.25) (layer B.Cu) (net 58))
   (segment (start 254.5 59.1) (end 262.237415 59.1) (width 0.25) (layer B.Cu) (net 58))
-  (segment (start 281.76252 80.15) (end 286.52504 80.15) (width 0.25) (layer B.Cu) (net 58))
-  (segment (start 213.5 80.15) (end 281.76252 80.15) (width 0.25) (layer B.Cu) (net 58))
+  (segment (start 213.5 80.15) (end 253.15 80.15) (width 0.25) (layer B.Cu) (net 58))
+  (segment (start 253.15 80.15) (end 255.5 77.8) (width 0.25) (layer B.Cu) (net 58))
+  (segment (start 255.5 77.8) (end 264.9 77.8) (width 0.25) (layer B.Cu) (net 58))
+  (segment (start 264.9 77.8) (end 267.3 80.2) (width 0.25) (layer B.Cu) (net 58))
+  (segment (start 267.3 80.2) (end 286.5 80.2) (width 0.25) (layer B.Cu) (net 58))
   (segment (start 128.74678 28.25764) (end 132.95764 28.25764) (width 0.25) (layer B.Cu) (net 59))
   (segment (start 134.2 29.5) (end 132.95764 28.25764) (width 0.25) (layer B.Cu) (net 59))
@@
   (segment (start 141.44686 87.94044) (end 141.44 87.9473) (width 0.25) (layer F.Cu) (net 74))
   (segment (start 141.44686 30.79764) (end 141.44686 87.94044) (width 0.25) (layer F.Cu) (net 74))
+  (segment (start 216.507405 96.01999) (end 206.08001 96.01999) (width 0.25) (layer B.Cu) (net 74))
+  (segment (start 206.08001 96.01999) (end 206.38001 96.01999) (width 0.25) (layer B.Cu) (net 74))
+  (segment (start 216.507405 96.01999) (end 216.507405 96.019991) (width 0.25) (layer B.Cu) (net 74))
+  (segment (start 216.507405 96.019991) (end 218.287414 97.8) (width 0.25) (layer B.Cu) (net 74))
+  (segment (start 223.7 97.8) (end 225.46999 99.56999) (width 0.25) (layer B.Cu) (net 74))
+  (segment (start 218.287414 97.8) (end 223.7 97.8) (width 0.25) (layer B.Cu) (net 74))
+  (segment (start 225.46999 99.56999) (end 255.23001 99.56999) (width 0.25) (layer B.Cu) (net 74))
+  (segment (start 255.23001 99.56999) (end 257 97.8) (width 0.25) (layer B.Cu) (net 74))
+  (segment (start 257 97.8) (end 257 91.9) (width 0.25) (layer B.Cu) (net 74))
+  (segment (start 161.31999 96.01999) (end 206.08001 96.01999) (width 0.25) (layer B.Cu) (net 74))
+  (segment (start 153.2473 87.9473) (end 161.31999 96.01999) (width 0.25) (layer B.Cu) (net 74))
+  (segment (start 141.44 87.9473) (end 153.2473 87.9473) (width 0.25) (layer B.Cu) (net 74))
   (segment (start 160.49694 27.22575) (end 160.49694 103.42607) (width 0.25) (layer F.Cu) (net 75))
   (segment (start 160.49625 60.80375) (end 160.49625 65.32591) (width 0.25) (layer B.Cu) (net 75))
@@
   (segment (start 216.35 96.4) (end 219.9 99.95) (width 0.25) (layer B.Cu) (net 90))
   (segment (start 178.15 96.4) (end 216.35 96.4) (width 0.25) (layer B.Cu) (net 90))
-  (segment (start 248.493972 99.95) (end 270.6 99.95) (width 0.25) (layer B.Cu) (net 90))
   (segment (start 219.9 99.95) (end 248.493972 99.95) (width 0.25) (layer B.Cu) (net 90))
   (segment (start 323.42504 96.75) (end 324.72504 98.05) (width 0.25) (layer B.Cu) (net 90))
@@
   (segment (start 255.68001 58.3) (end 256.1 58.71999) (width 0.25) (layer B.Cu) (net 90))
   (segment (start 254.5 58.3) (end 255.68001 58.3) (width 0.25) (layer B.Cu) (net 90))
+  (segment (start 253.15 99.95) (end 255.387415 99.95) (width 0.25) (layer B.Cu) (net 90))
+  (segment (start 248.493972 99.95) (end 253.15 99.95) (width 0.25) (layer B.Cu) (net 90))
+  (segment (start 262.6 92.737415) (end 262.6 83.6) (width 0.25) (layer B.Cu) (net 90))
+  (segment (start 262.6 83.6) (end 260.6 81.6) (width 0.25) (layer B.Cu) (net 90))
+  (segment (start 260.6 81.6) (end 260.6 80.1) (width 0.25) (layer B.Cu) (net 90))
+  (segment (start 267.1 99.95) (end 270.65 99.95) (width 0.25) (layer B.Cu) (net 90))
+  (segment (start 257.35 99.95) (end 256.368708 98.968708) (width 0.25) (layer B.Cu) (net 90))
+  (segment (start 267.1 99.95) (end 257.35 99.95) (width 0.25) (layer B.Cu) (net 90))
+  (segment (start 256.368708 98.968708) (end 262.6 92.737415) (width 0.25) (layer B.Cu) (net 90))
+  (segment (start 255.387415 99.95) (end 256.368708 98.968708) (width 0.25) (layer B.Cu) (net 90))
   (segment (start 257.31527 86.79725) (end 257.0323 86.79725) (width 0.25) (layer B.Cu) (net 91))
   (segment (start 260.66252 83.45) (end 257.31527 86.79725) (width 0.25) (layer B.Cu) (net 91))
-  (segment (start 261.61999 64.157404) (end 261.61999 72.042596) (width 0.25) (layer B.Cu) (net 92))
-  (segment (start 261.61999 72.042596) (end 260.152616 73.50997) (width 0.25) (layer B.Cu) (net 92))
-  (segment (start 260.522606 63.06002) (end 261.61999 64.157404) (width 0.25) (layer B.Cu) (net 92))
-  (segment (start 256.557405 63.06002) (end 260.522606 63.06002) (width 0.25) (layer B.Cu) (net 92))
-  (segment (start 255.717425 63.9) (end 256.557405 63.06002) (width 0.25) (layer B.Cu) (net 92))
-  (segment (start 254.5 63.9) (end 255.717425 63.9) (width 0.25) (layer B.Cu) (net 92))
-  (segment (start 256.034234 73.50997) (end 255.424264 72.9) (width 0.25) (layer B.Cu) (net 92))
-  (segment (start 255.424264 72.9) (end 255 72.9) (width 0.25) (layer B.Cu) (net 92))
-  (via (at 255 72.9) (size 0.6) (drill 0.3) (layers F.Cu B.Cu) (net 92))
-  (segment (start 260.152616 73.50997) (end 256.034234 73.50997) (width 0.25) (layer B.Cu) (net 92))
-  (segment (start 254.96252 89.72747) (end 257.0323 91.79725) (width 0.25) (layer F.Cu) (net 92))
-  (segment (start 254.96252 89.7) (end 254.96252 89.72747) (width 0.25) (layer F.Cu) (net 92))
-  (segment (start 254.78753 89.52501) (end 254.96252 89.7) (width 0.25) (layer F.Cu) (net 92))
-  (segment (start 255 72.9) (end 255 74.8) (width 0.25) (layer F.Cu) (net 92))
-  (segment (start 254.97506 74.8) (end 254.78753 74.98753) (width 0.25) (layer F.Cu) (net 92))
-  (segment (start 255 74.8) (end 254.97506 74.8) (width 0.25) (layer F.Cu) (net 92))
-  (segment (start 254.78753 74.98753) (end 254.78753 89.52501) (width 0.25) (layer F.Cu) (net 92))
   (zone (net 49) (net_name GND) (layer B.Cu) (hatch edge 0.508)
     (connect_pads (clearance 0.25))

Commit message: update plates
Parts:
- moved D61 3.46 mm to (261.3, 85.2)
- moved J1 2.38 mm to (250.0, 22.6)
- moved RCC1 2.38 mm to (241.8, 24.6)
- moved RCC2 2.38 mm to (257.8, 24.6)
Routing:
- net GND: track 16.4 -> 28.1 mm
- net ISP_RST: track 154.4 -> 157.4 mm
- net VBUS: track 22.2 -> 24.5 mm
- net DBUS-: track 14.8 -> 17.1 mm
- net DBUS+: track 13.8 -> 16.2 mm
- net row4: track 399.8 -> 397.8 mm
- net row3: track 407.8 -> 405.9 mm
- net D+: track 47.2 -> 48.9 mm
- net Enc0a: track 49.9 -> 51.1 mm
- net D-: track 48.0 -> 48.9 mm
- net Enc0b: track 53.0 -> 52.1 mm
Other:
- board size 264.3 x 111.6 mm -> 264.3 x 114 mm
- net class Default: via_dia 0.6 -> 0.65; via_drill 0.3 -> 0.35
- net class Power: via_dia 0.8 -> 0.9; via_drill 0.4 -> 0.5
- board text added: "niko rev 1.0 2021.10.31"

Commit message: new plates
Other:
- board text added: "niko rev 1.0 github.com/ricklicious"
- board text removed: "github.com/dierickdie niko rev 1.0"
Changed lines of the file:
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@@
   (gr_line (start 233.36348 129.77867) (end 266.70112 129.77867) (layer Edge.Cuts) (width 0.05))
   (gr_line (start 117.87237 27.38449) (end 117.87237 96.44103) (layer Edge.Cuts) (width 0.05))
-  (gr_text "github.com/dierickdie\nniko rev 1.0" (at 250.0323 123.82552) (layer B.SilkS)
+  (gr_text "niko rev 1.0\ngithub.com/ricklicious" (at 250.0323 123.82552) (layer B.SilkS)
     (effects (font (size 1.25 1.25) (thickness 0.2)) (justify mirror))
   )
