File: 03_bottom_plate/bottom_plate.kicad_pcb (KiCad board)
At the start: 2 copper layers, 257.2 x 112.5 mm, 71 parts, among them U1 HOLE, U10 HOLE, U11 HOLE, U12 HOLE, U13 HOLE, U14 HOLE, U15 HOLE, U16 HOLE, U17 HOLE, U18 HOLE, U19 HOLE, U2 HOLE, U20 HOLE, U21 HOLE, U22 HOLE, U23 HOLE, U24 HOLE, U25 HOLE, U26 HOLE, U27 HOLE, U28 HOLE, U29 HOLE, U3 HOLE, U30 HOLE, U31 HOLE, U32 HOLE, U33 HOLE, U34 HOLE, U35 HOLE, U36 HOLE, U37 HOLE, U38 HOLE, U39 HOLE, U4 HOLE, U40 HOLE, U41 HOLE, U42 HOLE, U43 HOLE, U44 HOLE, U45 HOLE, U46 HOLE, U47 HOLE, U48 HOLE, U49 HOLE, U5 HOLE, U50 HOLE, U51 HOLE, U52 HOLE, U53 HOLE, U54 HOLE, U55 HOLE, U56 HOLE, U57 HOLE, U58 HOLE, U59 HOLE, U6 HOLE, U60 HOLE, U61 HOLE, U7 HOLE, U8 HOLE, U9 HOLE

Commit message: remove 4 keys
Parts:
- removed R2: R_Small, Resistor_SMD:R_0805_2012Metric_Pad1.15x1.40mm_HandSolder
- removed U37, U38, U47, U48: HOLE, Keeb_footprints:MX100_outline
- added H9: MountingHole, MountingHole:MountingHole_3mm, F.Cu at (207.2, 89.3)
- moved H8 21.3 mm to (321.5, 158.9)
- moved H2 19.1 mm to (73.8, 158.9)
- moved H6 17.4 mm to (241.1, 178.0)
- moved R1 13.5 mm to (321.5, 100.0), turned to 180 degrees
- moved H7 9.53 mm to (321.5, 79.2)
- moved U11 9.53 mm to (302.4, 109.5)
- moved U23 9.53 mm to (302.4, 128.6)
- moved U35 9.53 mm to (302.4, 147.6)
- moved U59 9.53 mm to (302.4, 90.5)
- moved U21 9.53 mm to (264.3, 122.6)
- moved U33 9.53 mm to (264.3, 141.7)
- moved U44 9.53 mm to (238.1, 166.7)
- moved U45 9.53 mm to (264.3, 160.7)
- moved U57 9.53 mm to (264.3, 84.5)
- moved U9 9.53 mm to (264.3, 103.6)
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Routing:
- net GND: track 6.75 -> 1.51 mm
Other:
- board size 257.2 x 112.5 mm -> 266.7 x 118.2 mm

Commit message: update plates
Parts:
- added H10: MountingHole, random-keyboard-parts:Generic-Mounthole, F.Cu at (79.8, 78.0)
- added H11: MountingHole, random-keyboard-parts:Generic-Mounthole, F.Cu at (144.1, 73.2)
- added H12: MountingHole, random-keyboard-parts:Generic-Mounthole, F.Cu at (79.8, 158.9)
- added H13: MountingHole, random-keyboard-parts:Generic-Mounthole, F.Cu at (148.2, 176.2)
- added H14: MountingHole, random-keyboard-parts:Generic-Mounthole, F.Cu at (251.2, 73.2)
- added H15: MountingHole, random-keyboard-parts:Generic-Mounthole, F.Cu at (247.1, 176.2)
- added H16: MountingHole, random-keyboard-parts:Generic-Mounthole, F.Cu at (315.5, 78.0)
- added H17: MountingHole, random-keyboard-parts:Generic-Mounthole, F.Cu at (315.5, 158.9)
- R1: moved to F.Cu
- moved H1 0.60 mm to (73.8, 78.6)
- moved H7 0.60 mm to (321.5, 78.6)
Connections:
- R1 pad 2: (no net) -> Net-(R1-Pad2)
Other:
- board size 266.7 x 118.2 mm -> 266.7 x 117.9 mm
