File: 03.1_bottom_plate/top_plate.kicad_pcb (KiCad board)
At the start: 2 copper layers, 266.7 x 118.5 mm, 67 parts, among them U1 HOLE, U10 HOLE, U11 HOLE, U12 HOLE, U13 HOLE, U14 HOLE, U15 HOLE, U16 HOLE, U17 HOLE, U18 HOLE, U19 HOLE, U2 HOLE, U20 HOLE, U21 HOLE, U22 HOLE, U23 HOLE, U24 HOLE, U25 HOLE, U26 HOLE, U27 HOLE, U28 HOLE, U29 HOLE, U3 HOLE, U30 HOLE, U31 HOLE, U32 HOLE, U33 HOLE, U34 HOLE, U35 HOLE, U36 HOLE, U39 HOLE, U4 HOLE, U40 HOLE, U41 HOLE, U42 HOLE, U43 HOLE, U44 HOLE, U45 HOLE, U46 HOLE, U49 HOLE, U5 HOLE, U50 HOLE, U51 HOLE, U52 HOLE, U53 HOLE, U54 HOLE, U55 HOLE, U56 HOLE, U57 HOLE, U58 HOLE, U59 HOLE, U6 HOLE, U60 HOLE, U61 HOLE, U7 HOLE, U8 HOLE, U9 HOLE

Commit message: new plates
Other:
- board text added: "github.com/ricklicious"
- board text removed: "github.com/dierickdie"
Changed lines of the file:
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@@
     (effects (font (size 1 1) (thickness 0.15)))
   )
-  (gr_text github.com/dierickdie (at 197.645285 185.73771) (layer F.SilkS)
+  (gr_text github.com/ricklicious (at 197.645285 185.73771) (layer F.SilkS)
     (effects (font (size 1.25 1.25) (thickness 0.2)))
   )
